Commit message: bug fixes and first testing of hardware interface

File: description/urdf/test_state_publisher.urdf.xacro (robot description, xacro)
@@ -2,9 +2,9 @@
 <robot xmlns:xacro="http://www.ros.org/wiki/xacro" name="test_state_publisher_robot">
   <link name="base_link">
-    <inertial>
+    <!-- <inertial>
       <origin xyz="0 0 0" rpy="0 0 0"/>
       <mass value="3.0"/>
       <inertia ixx="0.001" ixy="0" ixz="0" iyy="0.001" iyz="0" izz="0.001"/>
-    </inertial>
+    </inertial> -->
     <visual name="Cube">
       <origin xyz="0 0 0" rpy="0 0 0"/>
@@ -15,9 +15,9 @@
   </link>
   <link name="link_1">
-    <inertial>
+    <!-- <inertial>
       <origin xyz="0 0 0" rpy="0 0 0"/>
       <mass value="3.0"/>
       <inertia ixx="0.001" ixy="0" ixz="0" iyy="0.001" iyz="0" izz="0.001"/>
-    </inertial>
+    </inertial> -->
     <visual name="Cube">
       <origin xyz="0 0 0" rpy="0 0 0"/>
@@ -54,22 +54,18 @@
       </hardware>
       <joint name="joint_1">
+          <param name="can_protocol">odrive</param>
+          <param name="can_id">1</param>
           <param name="can_channel">1</param>
-          <param name="can_id">1</param>
-          <param name="can_protocol">odrive</param>
-          <param name="position_scale">95.5</param>
-          <param name="velocity_scale">30.0</param>
-          <param name="effort_scale">18.0</param>
-          <param name="kp_scale">500.0</param>
-          <param name="kd_scale">5.0</param>
           <param name="axis_direction">-1</param>
+          <param name="position_offset">0.0</param>
           <param name="gear_ratio">1.0</param>
           <param name="torque_constant">0.0</param>
-          <param name="position_offset">0.0</param>
+          <param name="effort_max">1.0</param>
           <param name="position_min">-1.0</param>
           <param name="position_max">1.0</param>
           <param name="velocity_max">1.0</param>
-          <param name="effort_max">1.0</param>
           <param name="kp_max">1.0</param>
           <param name="kd_max">1.0</param>
+          <param name="ki_max">1.0</param>
           <param name="soft_start_duration_ms">0</param>
           <command_interface name="position"/>
@@ -78,4 +74,5 @@
           <command_interface name="kp"/>
           <command_interface name="kd"/>
+          <command_interface name="ki"/>
           <state_interface name="position"/>
           <state_interface name="velocity"/>

Commit message: Bug fixes to allow for multiple motors on same or multiple buses at up to 800Hz

File: description/urdf/test_state_publisher.urdf.xacro (robot description, xacro)
@@ -79,4 +79,30 @@
           <state_interface name="effort"/>
       </joint>
+      <joint name="joint_2">
+          <param name="can_protocol">odrive</param>
+          <param name="can_id">2</param>
+          <param name="can_channel">1</param>
+          <param name="axis_direction">-1</param>
+          <param name="position_offset">0.0</param>
+          <param name="gear_ratio">1.0</param>
+          <param name="torque_constant">0.09729</param>
+          <param name="effort_max">1.0</param>
+          <param name="position_min">-1.0</param>
+          <param name="position_max">1.0</param>
+          <param name="velocity_max">1.0</param>
+          <param name="kp_max">1.0</param>
+          <param name="kd_max">1.0</param>
+          <param name="ki_max">1.0</param>
+          <param name="soft_start_duration_ms">0</param>
+          <command_interface name="position"/>
+          <command_interface name="velocity"/>
+          <command_interface name="effort"/>
+          <command_interface name="kp"/>
+          <command_interface name="kd"/>
+          <command_interface name="ki"/>
+          <state_interface name="position"/>
+          <state_interface name="velocity"/>
+          <state_interface name="effort"/>
+      </joint>
       <sensor name="imu_sensor">
           <state_interface name="orientation.x"/>

Commit message: Tested feedback from 3 ODrives on 1 channel at 1kHz.

File: description/urdf/test_state_publisher.urdf.xacro (robot description, xacro)
@@ -105,4 +105,30 @@
           <state_interface name="effort"/>
       </joint>
+      <joint name="joint_3">
+          <param name="can_protocol">odrive</param>
+          <param name="can_id">3</param>
+          <param name="can_channel">1</param>
+          <param name="axis_direction">-1</param>
+          <param name="position_offset">0.0</param>
+          <param name="gear_ratio">1.0</param>
+          <param name="torque_constant">0.09729</param>
+          <param name="effort_max">1.0</param>
+          <param name="position_min">-1.0</param>
+          <param name="position_max">1.0</param>
+          <param name="velocity_max">1.0</param>
+          <param name="kp_max">1.0</param>
+          <param name="kd_max">1.0</param>
+          <param name="ki_max">1.0</param>
+          <param name="soft_start_duration_ms">0</param>
+          <command_interface name="position"/>
+          <command_interface name="velocity"/>
+          <command_interface name="effort"/>
+          <command_interface name="kp"/>
+          <command_interface name="kd"/>
+          <command_interface name="ki"/>
+          <state_interface name="position"/>
+          <state_interface name="velocity"/>
+          <state_interface name="effort"/>
+      </joint>
       <sensor name="imu_sensor">
           <state_interface name="orientation.x"/>

Commit message: initial debug of moteus actuator interface

File: description/urdf/test_state_publisher.urdf.xacro (robot description, xacro)
@@ -54,7 +54,7 @@
       </hardware>
       <joint name="joint_1">
-          <param name="can_protocol">odrive</param>
+          <param name="can_protocol">moteus</param>
           <param name="can_id">1</param>
-          <param name="can_channel">1</param>
+          <param name="can_channel">2</param>
           <param name="axis_direction">-1</param>
           <param name="position_offset">0.0</param>
@@ -79,5 +79,5 @@
           <state_interface name="effort"/>
       </joint>
-      <joint name="joint_2">
+      <!-- <joint name="joint_2">
           <param name="can_protocol">odrive</param>
           <param name="can_id">2</param>
@@ -130,5 +130,5 @@
           <state_interface name="velocity"/>
           <state_interface name="effort"/>
-      </joint>
+      </joint> -->
       <sensor name="imu_sensor">
           <state_interface name="orientation.x"/>
